Commit message: added more to robot state test, but no little checking of output, just warn output to inspect

File: test/two_links_moving_joint.urdf (robot description, URDF)
Before this commit: robot test_robot_moving_joint, 2 links, 1 joints
Joints:
- joint joint1: axis (none) -> 0 1 0; origin xyz=5 0 0 rpy=0 0 1.57 -> xyz=4.0 0 0 rpy=0 0 0
